Commit message: Adapt racecar to race on setup

File: racecar_description/urdf/macros.xacro (robot description, xacro)
@@ -30,5 +30,5 @@
                                               izz="4E-06" />
 </xacro:macro>
-<xacro:macro name="hokuyo_inertial_params">
+<xacro:macro name="camera_inertial_params">
   <origin xyz="0 0 0" rpy="0 0 0" />
   <mass value="0.130" />
@@ -92,4 +92,10 @@
   </geometry>
 </xacro:macro>
+<xacro:macro name="camera_geometry">
+  <origin xyz="0 0 0" rpy="0 0 0" />
+  <geometry>
+    <box size="0.030 0.030 0.030"/>
+  </geometry>
+</xacro:macro>
 <!-- transmission macros -->
 <xacro:macro name="wheel_transmission" params="name">

File: racecar_description/urdf/racecar.xacro (robot description, xacro)
@@ -145,6 +145,31 @@
   </joint>
   <xacro:wheel_transmission name="right_front_wheel" />
-  <!-- camera -->
-  <link name="ros_camera_link">
+  <!-- Add Hokuyo laser scanner -->
+  <link name="laser">
+    <inertial>
+      <xacro:hokuyo_inertial_params />
+    </inertial>
+    <collision>
+      <origin xyz="0 0 0" rpy="0 0 0"/>
+      <geometry>
+        <box size="0.1 0.1 0.1"/>
+      </geometry>
+    </collision>
+    <visual>
+      <origin xyz="0 0 0" rpy="0 0 0"/>
+      <geometry>
+        <mesh filename="package://racecar_description/meshes/hokuyo.dae"/>
+        <material name="grey" />
+      </geometry>
+    </visual>
+  </link>
+  <joint name="hokuyo_joint" type="fixed">
+    <origin xyz="0.265 0.0 0.075" rpy="0 0 0"/>
+    <parent link="chassis" />
+    <child link="laser" />
+    <axis xyz="0 0 1" />
+  </joint>
+  <!-- zed camera -->
+  <link name="zed_camera_link">
     <inertial>
       <mass value="1e-5" />
@@ -166,12 +191,12 @@
     </visual>
   </link>
-  <joint name="ros_camera_joint" type="fixed">
+  <joint name="zed_camera_joint" type="fixed">
     <origin xyz="0.390 0 0.04" rpy="0 0 0"/>
     <parent link="chassis"/>
-    <child link="ros_camera_link"/>
+    <child link="zed_camera_link"/>
     <axis xyz="0 0 1" />
     <!-- <limit lower="0.0" upper="0.0" effort="0.0" velocity="0.0" /> -->
   </joint>
-  <!-- camera lenses -->
+  <!-- zed camera lenses -->
   <!-- It seems these have to have a non-zero mass to have a camera attached? -->
   <link name="camera_link"><!-- this needs to match the name in zed_wrapper/zed_tf.launch -->
@@ -182,5 +207,5 @@
     </inertial>
   </link>
-  <link name="camera_right_link">
+  <link name="zed_camera_right_link">
     <inertial>
       <mass value="1e-5" />
@@ -189,14 +214,14 @@
     </inertial>
   </link>
-  <joint name="camera_left_joint" type="fixed">
+  <joint name="zed_camera_left_joint" type="fixed">
     <origin xyz="0 0.06 0" rpy="0 0 0"/>
-    <parent link="ros_camera_link"/>
+    <parent link="zed_camera_link"/>
     <child link="camera_link"/>
     <axis xyz="0 0 1" />
   </joint>
-  <joint name="camera_right_joint" type="fixed">
+  <joint name="zed_camera_right_joint" type="fixed">
     <origin xyz="0 -0.06 0" rpy="0 0 0"/>
-    <parent link="camera_link"/>
-    <child link="camera_right_link"/>
+    <parent link="zed_camera_link"/>
+    <child link="zed_camera_right_link"/>
     <axis xyz="0 0 1" />
   </joint>

File: racecar_description/urdf/racecar_raceon.xacro (robot description, xacro)
@@ -145,87 +145,26 @@
   </joint>
   <xacro:wheel_transmission name="right_front_wheel" />
-  <!-- Add Hokuyo laser scanner -->
-  <link name="laser">
+  <!-- camera -->
+  <link name="camera_link">
     <inertial>
-      <xacro:hokuyo_inertial_params />
+      <xacro:camera_inertial_params />
     </inertial>
     <collision>
-      <origin xyz="0 0 0" rpy="0 0 0"/>
-      <geometry>
-        <box size="0.1 0.1 0.1"/>
-      </geometry>
+      <xacro:camera_geometry />
     </collision>
     <visual>
-      <origin xyz="0 0 0" rpy="0 0 0"/>
-      <geometry>
-        <mesh filename="package://racecar_description/meshes/hokuyo.dae"/>
-        <material name="grey" />
-      </geometry>
-    </visual>
-  </link>
-  <joint name="hokuyo_joint" type="fixed">
-    <origin xyz="0.265 0.0 0.075" rpy="0 0 0"/>
-    <parent link="chassis" />
-    <child link="laser" />
-    <axis xyz="0 0 1" />
-  </joint>
-  <!-- zed camera -->
-  <link name="zed_camera_link">
-    <inertial>
-      <mass value="1e-5" />
-      <origin xyz="0 0 0" rpy="0 0 0"/>
-      <inertia ixx="1e-6" ixy="0" ixz="0" iyy="1e-6" iyz="0" izz="1e-6" />
-    </inertial>
-    <collision>
-      <origin xyz="0 0 0" rpy="0 0 0"/>
-      <geometry>
-        <box size="0.033 0.175 0.030"/>
-      </geometry>
-    </collision>
-    <visual>
-      <origin xyz="0 0 0" rpy="0 0 0"/>
-      <geometry>
-        <box size="0.033 0.175 0.030"/>
-      </geometry>
+      <xacro:camera_geometry />
       <material name="red"/>
     </visual>
   </link>
-  <joint name="zed_camera_joint" type="fixed">
-    <origin xyz="0.390 0 0.04" rpy="0 0 0"/>
+  <joint name="camera_link_joint" type="fixed">
+    <origin xyz="0.3 0 0.2" rpy="0 0.46 0"/>
     <parent link="chassis"/>
-    <child link="zed_camera_link"/>
+    <child link="camera_link"/>
     <axis xyz="0 0 1" />
     <!-- <limit lower="0.0" upper="0.0" effort="0.0" velocity="0.0" /> -->
   </joint>
-  <!-- zed camera lenses -->
-  <!-- It seems these have to have a non-zero mass to have a camera attached? -->
-  <link name="camera_link"><!-- this needs to match the name in zed_wrapper/zed_tf.launch -->
-    <inertial>
-      <mass value="1e-5" />
-      <origin xyz="0 0 0" rpy="0 0 0"/>
-      <inertia ixx="1e-6" ixy="0" ixz="0" iyy="1e-6" iyz="0" izz="1e-6" />
-    </inertial>
-  </link>
-  <link name="zed_camera_right_link">
-    <inertial>
-      <mass value="1e-5" />
-      <origin xyz="0 0 0" rpy="0 0 0"/>
-      <inertia ixx="1e-6" ixy="0" ixz="0" iyy="1e-6" iyz="0" izz="1e-6" />
-    </inertial>
-  </link>
-  <joint name="zed_camera_left_joint" type="fixed">
-    <origin xyz="0 0.06 0" rpy="0 0 0"/>
-    <parent link="zed_camera_link"/>
-    <child link="camera_link"/>
-    <axis xyz="0 0 1" />
-  </joint>
-  <joint name="zed_camera_right_joint" type="fixed">
-    <origin xyz="0 -0.06 0" rpy="0 0 0"/>
-    <parent link="zed_camera_link"/>
-    <child link="zed_camera_right_link"/>
-    <axis xyz="0 0 1" />
-  </joint>
   <!-- Add the remaining xacros -->
-  <xacro:include filename="$(find racecar_description)/urdf/racecar.gazebo" />
+  <xacro:include filename="$(find racecar_description)/urdf/racecar_raceon.gazebo" />
   <xacro:include filename="$(find racecar_description)/urdf/materials.xacro" />
 </robot>
