Commit message: Add raceon final track

File: racecar_description/urdf/racecar_raceon.xacro (robot description, xacro)
@@ -159,5 +159,5 @@
   </link>
   <joint name="camera_link_joint" type="fixed">
-    <origin xyz="0.3 0 0.2" rpy="0 0.46 0"/>
+    <origin xyz="0.3 0 0.2" rpy="0 0.26179939 0"/>
     <parent link="chassis"/>
     <child link="camera_link"/>

Commit message: Add race0

File: racecar_description/urdf/racecar_raceon.xacro (robot description, xacro)
@@ -159,5 +159,5 @@
   </link>
   <joint name="camera_link_joint" type="fixed">
-    <origin xyz="0.3 0 0.2" rpy="0 0.26179939 0"/>
+    <origin xyz="0.3 0 0.25" rpy="0 0.46 0"/>
     <parent link="chassis"/>
     <child link="camera_link"/>

Commit message: Tune model

File: racecar_description/urdf/racecar_raceon.xacro (robot description, xacro)
@@ -159,5 +159,5 @@
   </link>
   <joint name="camera_link_joint" type="fixed">
-    <origin xyz="0.3 0 0.25" rpy="0 0.46 0"/>
+    <origin xyz="0.3 0 0.1" rpy="0 0.78 0"/>
     <parent link="chassis"/>
     <child link="camera_link"/>

Commit message: Adjust model and add new tracks

File: racecar_description/urdf/racecar_raceon.xacro (robot description, xacro)
@@ -159,5 +159,5 @@
   </link>
   <joint name="camera_link_joint" type="fixed">
-    <origin xyz="0.3 0 0.1" rpy="0 0.78 0"/>
+    <origin xyz="0.31 0 0.25" rpy="0 0.78 0"/>
     <parent link="chassis"/>
     <child link="camera_link"/>

Commit message: Change dimension to fit raceon car

File: racecar_description/urdf/racecar_raceon.xacro (robot description, xacro)
@@ -39,5 +39,5 @@
   </link>
   <joint name="left_rear_wheel_joint" type="continuous">
-    <origin xyz="0 0.1 0" rpy="1.5708 0 0" />
+    <origin xyz="0 0.075 0" rpy="1.5708 0 0" />
     <parent link="chassis" />
     <child link="left_rear_wheel" />
@@ -60,5 +60,5 @@
   </link>
   <joint name="right_rear_wheel_joint" type="continuous">
-    <origin xyz="0 -0.1 0" rpy="1.5708 0 0" />
+    <origin xyz="0 -0.075 0" rpy="1.5708 0 0" />
     <parent link="chassis" />
     <child link="right_rear_wheel" />
@@ -78,5 +78,5 @@
   </link>
   <joint name="left_steering_hinge_joint" type="revolute">
-    <origin xyz="0.325 0.1 0" rpy="0 1.5708 0" />
+    <origin xyz="0.255 0.075 0" rpy="0 1.5708 0" />
     <parent link="chassis" />
     <child link="left_steering_hinge" />
@@ -96,5 +96,5 @@
   </link>
   <joint name="right_steering_hinge_joint" type="continuous">
-    <origin xyz="0.325 -0.1 0" rpy="0 1.5708 0" />
+    <origin xyz="0.255 -0.075 0" rpy="0 1.5708 0" />
     <parent link="chassis" />
     <child link="right_steering_hinge" />
@@ -159,5 +159,5 @@
   </link>
   <joint name="camera_link_joint" type="fixed">
-    <origin xyz="0.31 0 0.25" rpy="0 0.78 0"/>
+    <origin xyz="0.225 0 0.225" rpy="0 0.78 0"/>
     <parent link="chassis"/>
     <child link="camera_link"/>

Commit message: Change color of chassis

File: racecar_description/urdf/racecar_raceon.xacro (robot description, xacro)
@@ -7,5 +7,5 @@
     <visual>
       <xacro:chassis_geometry/>
-      <material name="blue" />
+      <material name="white" />
     </visual>
   </link>
