Commit message: Replace chassis by a simple box

File: racecar_description/urdf/macros_raceon.xacro (robot description, xacro)
@@ -39,7 +39,7 @@
 <!-- geometry macros -->
 <xacro:macro name="chassis_geometry">
-  <origin xyz="0 0 0" rpy="0 0 0" />
+  <origin xyz="0.115 0 0" rpy="0 0 0" />
   <geometry>
-    <mesh filename="package://racecar_description/meshes/chassis.STL" />
+    <box size="0.33 0.12 0.05"/>
   </geometry>
 </xacro:macro>

File: racecar_description/urdf/racecar_raceon.xacro (robot description, xacro)
@@ -1,5 +1,5 @@
 <?xml version="1.0"?>
 <robot name="racecar" xmlns:xacro="http://www.ros.org/wiki/xacro">
-  <xacro:include filename="$(find racecar_description)/urdf/macros.xacro" />
+  <xacro:include filename="$(find racecar_description)/urdf/macros_raceon.xacro" />
   <!-- Add chassis and it's inertia link -->
   <link name="base_link" />

Commit message: Modify wheel dimension and change color to grey

File: racecar_description/urdf/macros_raceon.xacro (robot description, xacro)
@@ -39,7 +39,7 @@
 <!-- geometry macros -->
 <xacro:macro name="chassis_geometry">
-  <origin xyz="0.115 0 0" rpy="0 0 0" />
+  <origin xyz="0.135 0 -0.01" rpy="0 0 0" />
   <geometry>
-    <box size="0.33 0.12 0.05"/>
+    <box size="0.30 0.06 0.02"/>
   </geometry>
 </xacro:macro>
@@ -47,5 +47,5 @@
   <origin xyz="0 0 0" rpy="0 0 0" />
   <geometry>
-    <mesh filename="package://racecar_description/meshes/left_rear_wheel.STL" />
+    <cylinder length="0.025" radius="0.03" />
   </geometry>
 </xacro:macro>
@@ -53,5 +53,5 @@
   <origin xyz="0 0 0" rpy="0 0 0" />
   <geometry>
-    <mesh filename="package://racecar_description/meshes/right_rear_wheel.STL" />
+    <cylinder length="0.025" radius="0.03" />
   </geometry>
 </xacro:macro>
@@ -59,5 +59,5 @@
   <origin xyz="0 0 0" rpy="0 0 0" />
   <geometry>
-    <mesh filename="package://racecar_description/meshes/left_front_wheel.STL" />
+    <cylinder length="0.025" radius="0.03" />
   </geometry>
 </xacro:macro>
@@ -65,5 +65,5 @@
   <origin xyz="0 0 0" rpy="0 0 0" />
   <geometry>
-    <mesh filename="package://racecar_description/meshes/right_front_wheel.STL" />
+    <cylinder length="0.025" radius="0.03" />
   </geometry>
 </xacro:macro>
@@ -83,5 +83,5 @@
   <origin xyz="0 0 -0.0225" rpy="0 0 0" />
   <geometry>
-    <cylinder length="0.045" radius="0.05" />
+    <cylinder length="0.025" radius="0.03" />
   </geometry>
 </xacro:macro>
@@ -89,5 +89,5 @@
   <origin xyz="0 0 0.0225" rpy="0 0 0" />
   <geometry>
-    <cylinder length="0.045" radius="0.05" />
+    <cylinder length="0.025" radius="0.03" />
   </geometry>
 </xacro:macro>
@@ -95,5 +95,5 @@
   <origin xyz="0 0 0" rpy="0 0 0" />
   <geometry>
-    <box size="0.030 0.030 0.030"/>
+    <box size="0.02 0.02 0.02"/>
   </geometry>
 </xacro:macro>

File: racecar_description/urdf/racecar_raceon.xacro (robot description, xacro)
@@ -32,5 +32,5 @@
     <visual>
       <xacro:left_rear_wheel_geometry />
-      <material name="black" />
+      <material name="grey" />
     </visual>
     <collision>robot
@@ -53,5 +53,5 @@
     <visual>
       <xacro:right_rear_wheel_geometry />
-      <material name="black" />
+      <material name="grey" />
     </visual>
     <collision>
@@ -110,5 +110,5 @@
     <visual>
       <xacro:left_front_wheel_geometry />
-      <material name="black" />
+      <material name="grey" />
     </visual>
     <collision>
@@ -131,5 +131,5 @@
     <visual>
       <xacro:right_front_wheel_geometry />
-      <material name="black" />
+      <material name="grey" />
     </visual>
     <collision>

Commit message: Adjuset frction parameters

File: racecar_description/urdf/macros_raceon.xacro (robot description, xacro)
@@ -81,5 +81,5 @@
 </xacro:macro>
 <xacro:macro name="left_wheels_collision_geometry">
-  <origin xyz="0 0 -0.0225" rpy="0 0 0" />
+  <origin xyz="0 0 0" rpy="0 0 0" />
   <geometry>
     <cylinder length="0.025" radius="0.03" />
@@ -87,5 +87,5 @@
 </xacro:macro>
 <xacro:macro name="right_wheels_collision_geometry">
-  <origin xyz="0 0 0.0225" rpy="0 0 0" />
+  <origin xyz="0 0 0" rpy="0 0 0" />
   <geometry>
     <cylinder length="0.025" radius="0.03" />

File: racecar_description/urdf/racecar_raceon.xacro (robot description, xacro)
@@ -34,5 +34,5 @@
       <material name="grey" />
     </visual>
-    <collision>robot
+    <collision>
       <xacro:left_wheels_collision_geometry />
     </collision>
